Commit message: added scripts for controller

File: Legged_robot/urdf/Legged_robot.urdf (robot description, URDF)
Before this commit: robot Legged_robot, 7 links, 6 joints
Links:
- removed link link_2_2
- added link link2_2, mass 7.58539816339745E-05; collision mesh filename=package://Legged_robot/meshes/link_2_2.STL; visual mesh filename=package://Legged_robot/meshes/link_2_2.STL
- link link_1_1: mass 8.78539816339741E-05 -> 8.78539816339742E-05
Joints:
- removed joint hip_link2_1
- added joint hip_link/_2_1: type revolute, parent hip, child link_2_1, origin xyz=-0.0056483 -0.0084654 0.034295 rpy=1.5708 -0.75702 0, axis 0 0 1, limit lower=0 upper=0 effort=0 velocity=0
- joint hip_link_2_2: child link_2_2 -> link2_2; limit (none) -> lower=0 upper=0 effort=0 velocity=0; origin xyz=-0.00564830078198353 -0.00146542786747287 0.0342954427878388 rpy=1.5707963267949 0 0 -> xyz=-0.0056483 -0.0014654 0.034295 rpy=1.5708 0 0; type continuous -> revolute
- joint link_1_1_foot_1: limit (none) -> lower=0 upper=0 effort=0 velocity=0; origin xyz=0 -0.014 0 rpy=0 0 0.00661019113303249 -> xyz=0 -0.014 0 rpy=0 0 0.6044; type continuous -> revolute
- joint link_1_2_foot_2: limit (none) -> lower=0 upper=0 effort=0 velocity=0; origin xyz=0 -0.014 0 rpy=0 0 0.0617710617631891 -> xyz=0 -0.014 0 rpy=0 0 0.061771; type continuous -> revolute
- joint link_2_1_link_1_1: limit (none) -> lower=0 upper=0 effort=0 velocity=0; origin xyz=0 -0.0140000000000002 0 rpy=0 0 -1.36435679641865 -> xyz=0 -0.014 0 rpy=0 0 -1.3614; type continuous -> revolute
- joint link_2_2_link_1_2: limit (none) -> lower=0 upper=0 effort=0 velocity=0; origin xyz=0 -0.014 0 rpy=0 0 -0.0617710617631891 -> xyz=0 -0.014 0 rpy=0 0 -0.061771; parent link_2_2 -> link2_2; type continuous -> revolute

Commit message: testing ik

File: Legged_robot/urdf/Legged_robot.urdf (robot description, URDF)
Before this commit: robot Legged_robot, 7 links, 6 joints
Joints:
- removed joint hip_link/_2_1
- added joint hip_link_2_1: type revolute, parent hip, child link_2_1, origin xyz=-0.0056483 -0.0084654 0.034295 rpy=1.5708 -0.75702 0, axis 0 0 1, limit lower=-1.57 upper=1.57 effort=10 velocity=3.14
- joint hip_link_2_2: limit lower=0 upper=0 effort=0 velocity=0 -> lower=-1.57 upper=1.57 effort=10 velocity=3.14
- joint link_1_1_foot_1: limit lower=0 upper=0 effort=0 velocity=0 -> lower=-1.57 upper=1.57 effort=10 velocity=3.14
- joint link_1_2_foot_2: limit lower=0 upper=0 effort=0 velocity=0 -> lower=-1.57 upper=1.57 effort=10 velocity=3.14
- joint link_2_1_link_1_1: limit lower=0 upper=0 effort=0 velocity=0 -> lower=-2.0944 upper=1.0472 effort=10 velocity=3.14
- joint link_2_2_link_1_2: limit lower=0 upper=0 effort=0 velocity=0 -> lower=-2.0944 upper=1.0472 effort=10 velocity=3.14
